File: electronics/Greenhouse_Climate_Sensor_V1_0.kicad_sch (KiCad schematic)
At the start: 12 parts, among them SW1 SW_SPST, U1 NodeMCU_1.0_(ESP-12E), U2 DHT22, U3 AMS1117-3.3

Commit message: goes to sleep for 60s after each measurement. Doesn't do anything if battery is low, checks after 1h.
Connections:
- net dht_data: now also U1.28 (D2(GPIO4)); no longer U1.27 (D3(GPIO0))
- net ~{rst}: now reaches U1.13 (RST)
- net ~{rst}: now also U1.30 (D0(GPIO16))
- no-connect marks 0 -> 19
Other:
- moved on the sheet: R3, U2
Changed lines of the file:
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@@
 (kicad_sch (version 20211123) (generator eeschema)
   (paper "A4")
-  (junction (at 160.02 62.23) (diameter 0) (color 0 0 0 0)
+  (junction (at 160.02 59.69) (diameter 0) (color 0 0 0 0)
   )
   (junction (at 181.61 109.22) (diameter 0) (color 0 0 0 0)
@@
   (junction (at 157.48 109.22) (diameter 0) (color 0 0 0 0)
   )
+  (no_connect (at 97.79 74.93))
+  (no_connect (at 138.43 72.39))
+  (no_connect (at 138.43 80.01))
+  (no_connect (at 138.43 74.93))
+  (no_connect (at 97.79 82.55))
+  (no_connect (at 97.79 62.23))
+  (no_connect (at 97.79 67.31))
+  (no_connect (at 97.79 64.77))
+  (no_connect (at 138.43 64.77))
+  (no_connect (at 179.07 62.23))
+  (no_connect (at 97.79 72.39))
+  (no_connect (at 138.43 82.55))
+  (no_connect (at 97.79 57.15))
+  (no_connect (at 138.43 62.23))
+  (no_connect (at 97.79 69.85))
+  (no_connect (at 138.43 85.09))
+  (no_connect (at 138.43 77.47))
+  (no_connect (at 97.79 59.69))
+  (no_connect (at 138.43 57.15))
   (wire (pts (xy 96.52 77.47) (xy 96.52 87.63))
     (stroke (width 0) (type default) (color 0 0 0 0))
@@
     (stroke (width 0) (type default) (color 0 0 0 0))
   )
-  (wire (pts (xy 160.02 60.96) (xy 160.02 62.23))
+  (wire (pts (xy 160.02 58.42) (xy 160.02 59.69))
     (stroke (width 0) (type default) (color 0 0 0 0))
   )
@@
     (stroke (width 0) (type default) (color 0 0 0 0))
   )
+  (wire (pts (xy 97.79 85.09) (xy 91.44 85.09))
+    (stroke (width 0) (type default) (color 0 0 0 0))
+  )
   (wire (pts (xy 138.43 69.85) (xy 139.7 69.85))
     (stroke (width 0) (type default) (color 0 0 0 0))
@@
     (stroke (width 0) (type default) (color 0 0 0 0))
   )
-  (wire (pts (xy 160.02 52.07) (xy 160.02 53.34))
+  (wire (pts (xy 160.02 49.53) (xy 160.02 50.8))
     (stroke (width 0) (type default) (color 0 0 0 0))
   )
@@
     (stroke (width 0) (type default) (color 0 0 0 0))
   )
-  (wire (pts (xy 160.02 62.23) (xy 165.1 62.23))
+  (wire (pts (xy 160.02 59.69) (xy 165.1 59.69))
     (stroke (width 0) (type default) (color 0 0 0 0))
   )
@@
     (stroke (width 0) (type default) (color 0 0 0 0))
   )
-  (wire (pts (xy 172.72 69.85) (xy 172.72 71.12))
+  (wire (pts (xy 172.72 67.31) (xy 172.72 68.58))
     (stroke (width 0) (type default) (color 0 0 0 0))
   )
@@
     (stroke (width 0) (type default) (color 0 0 0 0))
   )
-  (wire (pts (xy 138.43 62.23) (xy 160.02 62.23))
+  (wire (pts (xy 138.43 59.69) (xy 160.02 59.69))
     (stroke (width 0) (type default) (color 0 0 0 0))
   )
@@
     (stroke (width 0) (type default) (color 0 0 0 0))
   )
+  (wire (pts (xy 138.43 54.61) (xy 147.32 54.61))
+    (stroke (width 0) (type default) (color 0 0 0 0))
+  )
   (wire (pts (xy 204.47 109.22) (xy 204.47 110.49))
     (stroke (width 0) (type default) (color 0 0 0 0))
@@
     (stroke (width 0) (type default) (color 0 0 0 0))
   )
-  (wire (pts (xy 172.72 52.07) (xy 172.72 54.61))
+  (wire (pts (xy 172.72 49.53) (xy 172.72 52.07))
     (stroke (width 0) (type default) (color 0 0 0 0))
   )
@@
   (wire (pts (xy 181.61 109.22) (xy 181.61 110.49))
     (stroke (width 0) (type default) (color 0 0 0 0))
+  )
+  (label "~{rst}" (at 140.97 54.61 0)
+    (effects (font (size 1.27 1.27)) (justify left bottom))
   )
   (label "batt_direct" (at 133.35 109.22 0)
@@
     (effects (font (size 1.27 1.27)) (justify left bottom))
   )
-  (label "dht_data" (at 148.59 62.23 0)
+  (label "dht_data" (at 140.97 59.69 0)
+    (effects (font (size 1.27 1.27)) (justify left bottom))
+  )
+  (label "~{rst}" (at 91.44 85.09 0)
     (effects (font (size 1.27 1.27)) (justify left bottom))
   )
@@
     (pin "1")
   )
-  (symbol (lib_name "GND_1") (lib_id "power:GND") (at 172.72 71.12 0) (unit 1)
-    (in_bom yes) (on_board yes) (fields_autoplaced)
-    (property "Reference" "#PWR015" (id 0) (at 172.72 77.47 0)
-      (effects (font (size 1.27 1.27)) hide)
-    )
-    (property "Value" "GND" (id 1) (at 172.72 76.2 0))
-    (property "Footprint" "" (id 2) (at 172.72 71.12 0)
-      (effects (font (size 1.27 1.27)) hide)
-    )
-    (property "Datasheet" "" (id 3) (at 172.72 71.12 0)
+  (symbol (lib_name "GND_1") (lib_id "power:GND") (at 172.72 68.58 0) (unit 1)
+    (in_bom yes) (on_board yes) (fields_autoplaced)
+    (property "Reference" "#PWR015" (id 0) (at 172.72 74.93 0)
+      (effects (font (size 1.27 1.27)) hide)
+    )
+    (property "Value" "GND" (id 1) (at 172.72 73.66 0))
+    (property "Footprint" "" (id 2) (at 172.72 68.58 0)
+      (effects (font (size 1.27 1.27)) hide)
+    )
+    (property "Datasheet" "" (id 3) (at 172.72 68.58 0)
       (effects (font (size 1.27 1.27)) hide)
     )
@@
     (pin "3")
   )
-  (symbol (lib_id "power:+3.3V") (at 172.72 52.07 0) (unit 1)
-    (in_bom yes) (on_board yes) (fields_autoplaced)
-    (property "Reference" "#PWR014" (id 0) (at 172.72 55.88 0)
-      (effects (font (size 1.27 1.27)) hide)
-    )
-    (property "Value" "+3.3V" (id 1) (at 172.72 46.99 0))
-    (property "Footprint" "" (id 2) (at 172.72 52.07 0)
-      (effects (font (size 1.27 1.27)) hide)
-    )
-    (property "Datasheet" "" (id 3) (at 172.72 52.07 0)
+  (symbol (lib_id "power:+3.3V") (at 172.72 49.53 0) (unit 1)
+    (in_bom yes) (on_board yes) (fields_autoplaced)
+    (property "Reference" "#PWR014" (id 0) (at 172.72 53.34 0)
+      (effects (font (size 1.27 1.27)) hide)
+    )
+    (property "Value" "+3.3V" (id 1) (at 172.72 44.45 0))
+    (property "Footprint" "" (id 2) (at 172.72 49.53 0)
+      (effects (font (size 1.27 1.27)) hide)
+    )
+    (property "Datasheet" "" (id 3) (at 172.72 49.53 0)
       (effects (font (size 1.27 1.27)) hide)
     )
@@
     (pin "1")
   )
-  (symbol (lib_id "Sensor:DHT11") (at 172.72 62.23 0) (mirror y) (unit 1)
-    (in_bom yes) (on_board yes) (fields_autoplaced)
-    (property "Reference" "U2" (id 0) (at 179.07 60.9599 0)
+  (symbol (lib_id "Sensor:DHT11") (at 172.72 59.69 0) (mirror y) (unit 1)
+    (in_bom yes) (on_board yes) (fields_autoplaced)
+    (property "Reference" "U2" (id 0) (at 179.07 58.4199 0)
       (effects (font (size 1.27 1.27)) (justify right))
     )
-    (property "Value" "DHT22" (id 1) (at 179.07 63.4999 0)
+    (property "Value" "DHT22" (id 1) (at 179.07 60.9599 0)
       (effects (font (size 1.27 1.27)) (justify right))
     )
-    (property "Footprint" "Sensor:Aosong_DHT11_5.5x12.0_P2.54mm" (id 2) (at 172.72 72.39 0)
-      (effects (font (size 1.27 1.27)) hide)
-    )
-    (property "Datasheet" "http://akizukidenshi.com/download/ds/aosong/DHT11.pdf" (id 3) (at 168.91 55.88 0)
+    (property "Footprint" "Sensor:Aosong_DHT11_5.5x12.0_P2.54mm" (id 2) (at 172.72 69.85 0)
+      (effects (font (size 1.27 1.27)) hide)
+    )
+    (property "Datasheet" "http://akizukidenshi.com/download/ds/aosong/DHT11.pdf" (id 3) (at 168.91 53.34 0)
       (effects (font (size 1.27 1.27)) hide)
     )
@@
     (pin "1")
   )
-  (symbol (lib_id "Device:R") (at 160.02 57.15 0) (unit 1)
+  (symbol (lib_id "Device:R") (at 160.02 54.61 0) (unit 1)
     (in_bom yes) (on_board yes)
-    (property "Reference" "R3" (id 0) (at 162.56 55.8799 0)
-      (effects (font (size 1.27 1.27)) (justify left))
-    )
-    (property "Value" "10k" (id 1) (at 162.56 58.4199 0)
-      (effects (font (size 1.27 1.27)) (justify left))
-    )
-    (property "Footprint" "Resistor_THT:R_Axial_DIN0309_L9.0mm_D3.2mm_P2.54mm_Vertical" (id 2) (at 158.242 57.15 90)
-      (effects (font (size 1.27 1.27)) hide)
-    )
-    (property "Datasheet" "~" (id 3) (at 160.02 57.15 0)
+    (property "Reference" "R3" (id 0) (at 162.56 53.3399 0)
+      (effects (font (size 1.27 1.27)) (justify left))
+    )
+    (property "Value" "10k" (id 1) (at 162.56 55.8799 0)
+      (effects (font (size 1.27 1.27)) (justify left))
+    )
+    (property "Footprint" "Resistor_THT:R_Axial_DIN0309_L9.0mm_D3.2mm_P2.54mm_Vertical" (id 2) (at 158.242 54.61 90)
+      (effects (font (size 1.27 1.27)) hide)
+    )
+    (property "Datasheet" "~" (id 3) (at 160.02 54.61 0)
       (effects (font (size 1.27 1.27)) hide)
     )
@@
     (pin "2")
   )
-  (symbol (lib_id "power:+3.3V") (at 160.02 52.07 0) (unit 1)
-    (in_bom yes) (on_board yes) (fields_autoplaced)
-    (property "Reference" "#PWR012" (id 0) (at 160.02 55.88 0)
-      (effects (font (size 1.27 1.27)) hide)
-    )
-    (property "Value" "+3.3V" (id 1) (at 160.02 46.99 0))
-    (property "Footprint" "" (id 2) (at 160.02 52.07 0)
-      (effects (font (size 1.27 1.27)) hide)
-    )
-    (property "Datasheet" "" (id 3) (at 160.02 52.07 0)
-      (effects (font (size 1.27 1.27)) hide)
-    )
+  (symbol (lib_id "power:+3.3V") (at 160.02 49.53 0) (unit 1)
+    (in_bom yes) (on_board yes) (fields_autoplaced)
+    (property "Reference" "#PWR012" (id 0) (at 160.02 53.34 0)
+      (effects (font (size 1.27 1.27)) hide)
+    )
+    (property "Value" "+3.3V" (id 1) (at 160.02 44.45 0))
+    (property "Footprint" "" (id 2) (at 160.02 49.53 0)
+      (effects (font (size 1.27 1.27)) hide)
+    )
+    (property "Datasheet" "" (id 3) (at 160.02 49.53 0)
+      (effects (font (size 1.27 1.27)) hide)
+    )
