File: electronics/Greenhouse_Climate_Sensor_V1_0.kicad_sch (KiCad schematic)
At the start: 12 parts, among them SW1 SW_SPST, U1 NodeMCU_1.0_(ESP-12E), U2 DHT22, U3 AMS1117-3.3

Commit message: main.cpp: open hotspot if button is pressed during startup
Parts:
- removed C2, C3: 22µF, Capacitor_SMD:C_1210_3225Metric_Pad1.33x2.70mm_HandSolder, symbol Device:C
- removed U3: AMS1117-3.3, Package_TO_SOT_SMD:SOT-223-3_TabPin2, symbol Regulator_Linear:AMS1117-3.3
- added SW?: SW_SPST, symbol Switch:SW_SPST
Connections:
- net GND: now also SW?.2 (B)
- net ~{open_hotspot}: now reaches U1.21 (D7(GPIO13))
- net ~{open_hotspot}: now also SW?.1 (A)
- no-connect marks 19 -> 18
Other:
- note added: "Buck Converter module based on TPS62827"
